File: smartportsd-nano-shield.sch (KiCad schematic (older format))
At the start: 18 parts, among them J1 DB25_Female_MountingHoles, J2 Conn_01x09, SW1 EJECT

Commit message: Add some docs
Parts:
- C1: Comment (none) -> Optional, 5V bulk for board
- D1, D2, D3, D4: Comment (none) -> Green
- D5: Comment (none) -> Red
- MOD1: Comment (none) -> From eBay/Aliexpress
- R2, R3, R4, R5: Comment (none) -> For active partition LED's
- R6: Comment (none) -> For status LED
Changed lines of the file:
@@
 F 2 "CARD-SD-ADAPTER-CATALEX:Catalex-MicroSD-Card-Down" H 6950 4350 50  0001 L BNN
 F 3 "" H 6950 4350 50  0001 L BNN
+F 4 "From eBay/Aliexpress" H 6950 4350 50  0001 C CNN "Comment"
 	1    6950 4350
 	1    0    0    -1
@@
 F 2 "LED_THT:LED_D5.0mm" H 4400 5100 50  0001 C CNN
 F 3 "~" H 4400 5100 50  0001 C CNN
+F 4 "Red" H 4400 5100 50  0001 C CNN "Comment"
 	1    4400 5100
 	-1   0    0    1
@@
 F 2 "Resistor_THT:R_Axial_DIN0207_L6.3mm_D2.5mm_P7.62mm_Horizontal" V 4630 5100 50  0001 C CNN
 F 3 "~" H 4700 5100 50  0001 C CNN
+F 4 "For status LED" H 4700 5100 50  0001 C CNN "Comment"
 	1    4700 5100
 	0    1    1    0
@@
 F 2 "LED_THT:LED_D5.0mm" H 4400 3650 50  0001 C CNN
 F 3 "~" H 4400 3650 50  0001 C CNN
+F 4 "Green" H 4400 3650 50  0001 C CNN "Comment"
 	1    4400 3650
 	-1   0    0    1
@@
 F 2 "Resistor_THT:R_Axial_DIN0207_L6.3mm_D2.5mm_P7.62mm_Horizontal" V 4630 3650 50  0001 C CNN
 F 3 "~" H 4700 3650 50  0001 C CNN
+F 4 "For active partition LED's" H 4700 3650 50  0001 C CNN "Comment"
 	1    4700 3650
 	0    1    1    0
@@
 F 2 "LED_THT:LED_D5.0mm" H 4400 4000 50  0001 C CNN
 F 3 "~" H 4400 4000 50  0001 C CNN
+F 4 "Green" H 4400 4000 50  0001 C CNN "Comment"
 	1    4400 4000
 	-1   0    0    1
@@
 F 2 "Resistor_THT:R_Axial_DIN0207_L6.3mm_D2.5mm_P7.62mm_Horizontal" V 4630 4000 50  0001 C CNN
 F 3 "~" H 4700 4000 50  0001 C CNN
+F 4 "For active partition LED's" H 4700 4000 50  0001 C CNN "Comment"
 	1    4700 4000
 	0    1    1    0
@@
 F 2 "LED_THT:LED_D5.0mm" H 4400 4350 50  0001 C CNN
 F 3 "~" H 4400 4350 50  0001 C CNN
+F 4 "Green" H 4400 4350 50  0001 C CNN "Comment"
 	1    4400 4350
 	-1   0    0    1
@@
 F 2 "Resistor_THT:R_Axial_DIN0207_L6.3mm_D2.5mm_P7.62mm_Horizontal" V 4630 4350 50  0001 C CNN
 F 3 "~" H 4700 4350 50  0001 C CNN
+F 4 "For active partition LED's" H 4700 4350 50  0001 C CNN "Comment"
 	1    4700 4350
 	0    1    1    0
@@
 F 2 "LED_THT:LED_D5.0mm" H 4400 4700 50  0001 C CNN
 F 3 "~" H 4400 4700 50  0001 C CNN
+F 4 "Green" H 4400 4700 50  0001 C CNN "Comment"
 	1    4400 4700
 	-1   0    0    1
@@
 F 2 "Resistor_THT:R_Axial_DIN0207_L6.3mm_D2.5mm_P7.62mm_Horizontal" V 4630 4700 50  0001 C CNN
 F 3 "~" H 4700 4700 50  0001 C CNN
+F 4 "For active partition LED's" H 4700 4700 50  0001 C CNN "Comment"
 	1    4700 4700
 	0    1    1    0
@@
 F 2 "Capacitor_THT:CP_Radial_D4.0mm_P1.50mm" H 7350 2750 50  0001 C CNN
 F 3 "~" H 7350 2750 50  0001 C CNN
+F 4 "Optional, 5V bulk for board" H 7350 2750 50  0001 C CNN "Comment"
 	1    7350 2750
 	1    0    0    -1
